File: src/board/openhome-board.sch (KiCad schematic (older format))
At the start: 11 parts, among them J1 Conn_01x03, J2 Conn_02x11_Odd_Even, J3 Conn_01x04, J4 Conn_01x02, J5 Conn_01x04, K1 G5Q-1, Q1 2N2219

Commit message: correct some comments + board
Parts:
- removed J5: Conn_01x04, atmo:POWER_UNIT, symbol Conn_01x04
- removed K1: G5Q-1, Relays_THT:Relay_SPDT_OMRON-G5Q, symbol G5Q-1
- added K1: SANYOU_SRD_Form_C, Relays_THT:Relay_SPDT_SANYOU_SRD_Series_Form_C, symbol SANYOU_SRD_Form_C
- J4: footprint Connectors:bornier2 -> (none)
Connections:
- net AC_L is gone; now on net +3V3: J4.1 (Pin_1)
- net AC_N is gone; now on net GND: J4.2 (Pin_2)
- net +3V3: now also K1.5
- net at D1.2 (A), Q1.3 (C): now also K1.2
- net at J1.3 (Pin_3): now also K1.3
- net at J1.1 (Pin_1): now also K1.4
- net at J1.2 (Pin_2): now also K1.1
- no-connect marks 1 -> 0
Changed lines of the file:
@@
 L GND #PWR01
 U 1 1 5AE78B5D
-P 8250 2400
-F 0 "#PWR01" H 8250 2150 50  0001 C CNN
-F 1 "GND" H 8250 2250 50  0000 C CNN
-F 2 "" H 8250 2400 50  0001 C CNN
-F 3 "" H 8250 2400 50  0001 C CNN
-	1    8250 2400
-	1    0    0    -1
-$EndComp
-$Comp
-L Conn_01x02 J4
-U 1 1 5AE78C12
-P 7400 2200
-F 0 "J4" H 7400 2300 50  0000 C CNN
-F 1 "Conn_01x02" H 7400 2000 50  0000 C CNN
-F 2 "Connectors:bornier2" H 7400 2200 50  0001 C CNN
-F 3 "" H 7400 2200 50  0001 C CNN
-	1    7400 2200
-	-1   0    0    1
+P 7000 2150
+F 0 "#PWR01" H 7000 1900 50  0001 C CNN
+F 1 "GND" H 7000 2000 50  0000 C CNN
+F 2 "" H 7000 2150 50  0001 C CNN
+F 3 "" H 7000 2150 50  0001 C CNN
+	1    7000 2150
+	1    0    0    -1
 $EndComp
 $Comp
 L +3.3V #PWR02
 U 1 1 5AE78DA7
-P 8050 2300
-F 0 "#PWR02" H 8050 2150 50  0001 C CNN
-F 1 "+3.3V" H 8050 2440 50  0000 C CNN
-F 2 "" H 8050 2300 50  0001 C CNN
-F 3 "" H 8050 2300 50  0001 C CNN
-	1    8050 2300
+P 6800 2050
+F 0 "#PWR02" H 6800 1900 50  0001 C CNN
+F 1 "+3.3V" H 6800 2190 50  0000 C CNN
+F 2 "" H 6800 2050 50  0001 C CNN
+F 3 "" H 6800 2050 50  0001 C CNN
+	1    6800 2050
 	-1   0    0    1
 $EndComp
@@
 Text GLabel 6750 1600 2    60   Input ~ 0
 I2C_THR_SDL
-Wire Wire Line
-	6250 1500 6750 1500
-Wire Wire Line
-	6250 1600 6750 1600
 $Comp
 L R R2
@@
 	1    0    0    -1
 $EndComp
-Wire Wire Line
-	6400 1050 6400 1500
-Connection ~ 6400 1500
-Wire Wire Line
-	6600 1050 6600 1600
-Connection ~ 6600 1600
-Wire Wire Line
-	6400 750  6600 750
 $Comp
 L +3.3V #PWR05
@@
 	1    0    0    -1
 $EndComp
-Connection ~ 6500 750
 $Comp
 L +3.3V #PWR06
@@
 	0    1    1    0
 $EndComp
-Wire Wire Line
-	2350 2650 2450 2650
-$Comp
-L G5Q-1 K1
-U 1 1 5AE7972B
-P 3150 2150
-F 0 "K1" H 3800 2500 50  0000 L CNN
-F 1 "G5Q-1" H 3800 2400 50  0000 L CNN
-F 2 "Relays_THT:Relay_SPDT_OMRON-G5Q" H 3800 2300 50  0001 L CNN
-F 3 "" H 3800 2000 50  0001 L CNN
-	1    3150 2150
-	1    0    0    -1
-$EndComp
 $Comp
 L 1N4001 D1
@@
 	0    1    1    0
 $EndComp
-Wire Wire Line
-	2750 1800 2750 1600
-Wire Wire Line
-	2750 1600 3150 1600
-Wire Wire Line
-	3150 1600 3150 1650
-Wire Wire Line
-	3150 2250 3150 2300
-Wire Wire Line
-	3150 2300 2750 2300
-Wire Wire Line
-	2750 2100 2750 2450
-Connection ~ 2750 2300
 $Comp
 L GND #PWR08
@@
 	1    0    0    -1
 $EndComp
-Connection ~ 2750 1600
 Text GLabel 1950 2650 0    60   Input ~ 0
 RELAY_DRV
 Text GLabel 5650 1400 0    60   Input ~ 0
 RELAY_DRV
-Wire Wire Line
-	5650 1400 5750 1400
-Wire Wire Line
-	1950 2650 2050 2650
 $Comp
 L Conn_01x03 J1
@@
 $EndComp
 $Comp
-L Conn_01x04 J5
-U 1 1 5AE89F6F
-P 8600 2200
-F 0 "J5" H 8600 2400 50  0000 C CNN
-F 1 "Conn_01x04" H 8600 1900 50  0000 C CNN
-F 2 "atmo:POWER_UNIT" H 8600 2200 50  0001 C CNN
-F 3 "" H 8600 2200 50  0001 C CNN
-	1    8600 2200
-	1    0    0    -1
-$EndComp
-Text GLabel 8350 2100 0    60   Input ~ 0
-AC_L
-Text GLabel 8350 2200 0    60   Input ~ 0
-AC_N
-Wire Wire Line
-	8350 2100 8400 2100
-Wire Wire Line
-	8350 2200 8400 2200
-Wire Wire Line
-	8050 2300 8400 2300
-Wire Wire Line
-	8250 2400 8400 2400
-Text GLabel 7600 2200 2    60   Input ~ 0
-AC_L
-Text GLabel 7600 2100 2    60   Input ~ 0
-AC_N
+L Conn_01x02 J4
+U 1 1 5AEF1FCE
+P 7350 2050
+F 0 "J4" H 7350 2150 50  0000 C CNN
+F 1 "Conn_01x02" H 7350 1850 50  0000 C CNN
+F 2 "" H 7350 2050 50  0001 C CNN
+F 3 "" H 7350 2050 50  0001 C CNN
+	1    7350 2050
+	1    0    0    -1
+$EndComp
+Wire Wire Line
+	6250 1500 6750 1500
+Wire Wire Line
+	6250 1600 6750 1600
+Wire Wire Line
+	6400 1050 6400 1500
+Connection ~ 6400 1500
+Wire Wire Line
+	6600 1050 6600 1600
+Connection ~ 6600 1600
+Wire Wire Line
+	6400 750  6600 750
+Connection ~ 6500 750
+Wire Wire Line
+	2350 2650 2450 2650
+Wire Wire Line
+	2750 1800 2750 1600
+Wire Wire Line
+	2750 1600 3150 1600
+Wire Wire Line
+	3150 1600 3150 1650
+Wire Wire Line
+	3150 2250 3150 2300
+Wire Wire Line
+	3150 2300 2750 2300
+Wire Wire Line
+	2750 2100 2750 2450
+Connection ~ 2750 2300
+Connection ~ 2750 1600
+Wire Wire Line
+	5650 1400 5750 1400
+Wire Wire Line
+	1950 2650 2050 2650
+Wire Wire Line
+	6800 2050 7150 2050
+Wire Wire Line
+	7000 2150 7150 2150
 Wire Wire Line
 	3650 1650 3650 1600
 Wire Wire Line
+	4250 1600 4250 1850
+Wire Wire Line
 	3650 1600 4250 1600
-Wire Wire Line
-	4250 1600 4250 1850
-Wire Wire Line
-	3550 2250 4250 2250
-Wire Wire Line
-	4250 2250 4250 2050
-NoConn ~ 4250 1950
+$Comp
+L SANYOU_SRD_Form_C K1
+U 1 1 5AEF2DC4
+P 3350 1950
+F 0 "K1" H 3800 2100 50  0000 L CNN
+F 1 "SANYOU_SRD_Form_C" H 3800 2000 50  0000 L CNN
+F 2 "Relays_THT:Relay_SPDT_SANYOU_SRD_Series_Form_C" H 4800 1900 50  0001 C CNN
+F 3 "" H 3350 1950 50  0001 C CNN
+	1    3350 1950
+	1    0    0    -1
+$EndComp
+Wire Wire Line
+	4250 2050 4100 2050
+Wire Wire Line
+	4100 2050 4100 1500
+Wire Wire Line
+	4100 1500 3450 1500
+Wire Wire Line
+	3450 1500 3450 1650
+Wire Wire Line
+	3550 2250 4000 2250
+Wire Wire Line
+	4000 2250 4000 1950
+Wire Wire Line
+	4000 1950 4250 1950
 $EndSCHEMATC
